Commit message: 基本知道了编写的规则，编辑了一部分内容

File: supervised learning/bipedRobotOne.urdf (robot description, URDF)
Before this commit: robot biped-one, 2 links, 0 joints
Links:
- removed link torso
- added link left-thigh, mass 2.0; collision box size=0.05 0.05 0.5; visual box size=0.05 0.05 0.5
- added link torso-base, mass 20; collision box size=0.12 0.25 0.4; visual box size=0.12 0.25 0.4
- link left-block: mass None -> 0.5; geometry collision box size=0.06 0.06 0.06; visual box size=0.06 0.06 0.06
Joints:
- added joint left_j1: type continuous, parent torso-base, child left-block, origin xyz=0 0.12 -0.2 rpy=0 0 0, axis 1 0 0, limit effort=100 velocity=100
- added joint left_j2: type continuous, parent left-block, child left-thigh, origin xyz=0 0 0 rpy=0 0 0, axis 0 1 0, limit effort=100 velocity=100

Commit message: 编写完一般的urdf模型，还有一点没明白的~

File: supervised learning/bipedRobotOne.urdf (robot description, URDF)
Before this commit: robot biped-one, 3 links, 2 joints
Links:
- added link left-foot, mass 0.1; collision sphere radius=0.025; visual sphere radius=0.025
- added link left-shank, mass 2.0; collision box size=0.05 0.05 0.5; visual box size=0.05 0.05 0.5
Joints:
- added joint left_j3: type continuous, parent left-thigh, child left-shank, origin xyz=0 0 -0.5 rpy=0 0 0, axis 0 1 0, limit effort=100 velocity=100
- added joint left_j4: type fixed, parent left-shank, child left-foot, origin xyz=0 0 -0.5 rpy=0 0 0

Commit message: 编写完成一个模型

File: supervised learning/bipedRobotOne.urdf (robot description, URDF)
Before this commit: robot biped-one, 5 links, 4 joints
Links:
- added link right-block, mass 0.5; collision box size=0.06 0.06 0.06; visual box size=0.06 0.06 0.06
- added link right-foot, mass 0.1; collision sphere radius=0.025; visual sphere radius=0.025
- added link right-shank, mass 2.0; collision box size=0.05 0.05 0.5; visual box size=0.05 0.05 0.5
- added link right-thigh, mass 2.0; collision box size=0.05 0.05 0.5; visual box size=0.05 0.05 0.5
Joints:
- added joint right_j1: type continuous, parent torso-base, child right-block, origin xyz=0 -0.12 -0.2 rpy=0 0 0, axis 1 0 0, limit effort=100 velocity=100
- added joint right_j2: type continuous, parent right-block, child right-thigh, origin xyz=0 0 0 rpy=0 0 0, axis 0 1 0, limit effort=100 velocity=100
- added joint right_j3: type continuous, parent right-thigh, child right-shank, origin xyz=0 0 -0.5 rpy=0 0 0, axis 0 1 0, limit effort=100 velocity=100
- added joint right_j4: type fixed, parent right-shank, child right-foot, origin xyz=0 0 -0.5 rpy=0 0 0

Commit message: 完成对关节的控制测试

File: supervised learning/bipedRobotOne.urdf (robot description, URDF)
Before this commit: robot biped-one, 9 links, 8 joints
Links:
- link torso-base: mass 20 -> 0

Commit message: 编辑了控制的很少一部分

File: supervised learning/bipedRobotOne.urdf (robot description, URDF)
Before this commit: robot biped-one, 9 links, 8 joints
Links:
- link torso-base: mass 0 -> 20
